Commit message: Mandamo tudo

File: remy_ws/src/urdf2_description/urdf/urdf2.xacro (robot description, xacro)
@@ -24,5 +24,5 @@
   </collision>
 </link>
-<link name="limb2_v1_1">
+<link name="laser_link">
   <inertial>
     <origin xyz="-0.02149999999999923 -0.023058640719597706 0.016872379763677364" rpy="0 0 0"/>
@@ -64,18 +64,4 @@
   </collision>s
 </link>
-<link name="realsense_link">
-  <visual>
-    <origin xyz="0 0 0" rpy="0 0 0"/>
-    <geometry>
-      <box size="0.05 0.05 0.02"/>
-    </geometry>
-    <material name="black"/>
-  </visual>
-</link>
-<joint name="realsense_joint" type="fixed">
-  <origin xyz="0 0 0" rpy="0 0 0"/>
-  <parent link="limb3_v1_1"/>
-  <child link="realsense_link"/>
-</joint>
 <link name="limb1_v1_1">
   <inertial>
@@ -278,11 +264,11 @@
   </collision>
 </link>
-<joint name="rig2" type="fixed">
-  <origin xyz="0.0215 -0.190948 0.125363" rpy="0 0 0"/>
-  <parent link="base_link"/>
-  <child link="limb2_v1_1"/>
+<joint name="laser_joint" type="fixed">
+  <origin xyz="0.0215 -0.190948 0.125363" rpy="0 0 -1.5708"/>
+  <parent link="base_link"/>
+  <child link="laser_link"/>
 </joint>
 <joint name="rig3" type="fixed">
-  <origin xyz="0.0325 0.0265 1.500001" rpy="0 0 0"/>
+  <origin xyz="0.0325 0.0265 1.500001" rpy="0 0 -1.5708"/>
   <parent link="base_link"/>
   <child link="limb3_v1_1"/>
@@ -292,5 +278,5 @@
   <parent link="base_link"/>
   <child link="limb1_v1_1"/>
-  <axis xyz="-1.0 -0.0 -0.0"/>
+  <axis xyz="1 0 0" rpy="0 0 0"/> <!-- roda direita gira no eixo Y -->
 </joint>
 <joint name="rev2" type="continuous">
@@ -298,5 +284,5 @@
   <parent link="base_link"/>
   <child link="limb1_v1__1__1"/>
-  <axis xyz="1.0 0.0 -0.0"/>
+  <axis xyz="1 0 0" rpy="0 0 0"/> <!-- roda esquerda gira no eixo Y -->
 </joint>
 <joint name="rev11" type="continuous">

Commit message: Tamo quase la

File: remy_ws/src/urdf2_description/urdf/urdf2.xacro (robot description, xacro)
@@ -4,4 +4,10 @@
 <xacro:include filename="$(find urdf2_description)/urdf/urdf2.trans" />
 <xacro:include filename="$(find urdf2_description)/urdf/urdf2.gazebo" />
+<link name="base_footprint"/>
+<joint name="base_joint" type="fixed">
+  <parent link="base_footprint"/>
+  <child link="base_link"/>
+  <origin xyz="0 0 0" rpy="0 0 0"/>
+</joint>
 <link name="base_link">
   <inertial>
@@ -24,5 +30,5 @@
   </collision>
 </link>
-<link name="laser_link">
+<link name="laser">
   <inertial>
     <origin xyz="-0.02149999999999923 -0.023058640719597706 0.016872379763677364" rpy="0 0 0"/>
@@ -267,5 +273,5 @@
   <origin xyz="0.0215 -0.190948 0.125363" rpy="0 0 -1.5708"/>
   <parent link="base_link"/>
-  <child link="laser_link"/>
+  <child link="laser"/>
 </joint>
 <joint name="rig3" type="fixed">
